Commit message: first step to gazebo support
rename links and joints to have semantic names
add inertia to all links
add laser and diffdrive plugins

Signed-off-by: Mikael Arguedas <mikael.arguedas@gmail.com>

File: confbot_description/urdf/confbot.urdf (robot description, URDF)
Before this commit: robot confbot, 4 links, 3 joints
Links:
- removed link laser_link
- added link caster_wheel_front_link, mass 1; collision sphere radius=0.05; visual sphere radius=0.05
- added link caster_wheel_rear_link, mass 1; collision sphere radius=0.05; visual sphere radius=0.05
- added link laser_frame, mass 1; collision box size=0.1 0.1 0.1; visual box size=0.1 0.1 0.1
- link base_link: mass None -> 5; geometry collision box size=1 1 0.1; visual mesh filename=file:///media/mikatchou/ROS/ros2/roscon2019/roscon2019_ws/i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
- link wheel_l_link: mass None -> 1; geometry collision cylinder length=0.05 radius=0.1; visual cylinder length=0.05 radius=0.1
- link wheel_r_link: mass None -> 1; geometry collision cylinder length=0.05 radius=0.1; visual cylinder length=0.05 radius=0.1
Joints:
- removed joint wheel_l_frame
- removed joint wheel_r_frame
- added joint caster_wheel_front_joint: type continuous, parent base_link, child caster_wheel_front_link, origin xyz=0.4 0.0 -0.05 rpy=0 0 0, axis 1.0 1.0 0
- added joint caster_wheel_rear_joint: type continuous, parent base_link, child caster_wheel_rear_link, origin xyz=-0.4 0.0 -0.05 rpy=0 0 0, axis 1.0 1.0 0
- added joint wheel_l_joint: type continuous, parent base_link, child wheel_l_link, origin xyz=0 0.55 0.0 rpy=0 0 0, axis 0 1.0 0
- added joint wheel_r_joint: type continuous, parent base_link, child wheel_r_link, origin xyz=0 -0.55 0.0 rpy=0 0 0, axis 0 1.0 0
- joint laser_frame: child laser_link -> laser_frame

Commit message: restore package:// path
Signed-off-by: Mikael Arguedas <mikael.arguedas@gmail.com>

File: confbot_description/urdf/confbot.urdf (robot description, URDF)
Before this commit: robot confbot, 6 links, 5 joints
Links:
- link base_link: geometry collision box size=1 1 0.1; visual mesh filename=package://confbot_description/meshes/confbot.dae
